File: daughter_board.sch (KiCad schematic (older format))
At the start: 4 parts, among them J1 Xplained_Pro_Extension_Header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, J2 Xplained_Pro_Extension_Header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, J3 Xplained_Pro_Extension_Header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, U1 ms5611

Commit message: Add preliminary footprint associations
Parts:
- J1, J2, J3: footprint (none) -> Socket_Strips:Socket_Strip_Angled_2x10_Pitch2.54mm
- U1: footprint (none) -> Housings_LGA:LGA-8_3x5mm_Pitch1.25mm
Changed lines of the file:
@@
 F 0 "U1" H 5975 3100 60  0000 C CNN
 F 1 "ms5611" H 5550 3600 60  0000 C CNN
-F 2 "" H 5575 3725 60  0001 C CNN
+F 2 "Housings_LGA:LGA-8_3x5mm_Pitch1.25mm" H 5575 3725 60  0001 C CNN
 F 3 "" H 5575 3725 60  0001 C CNN
 	1    5550 3600
@@
 F 0 "J1" H 3050 3800 50  0000 C CNN
 F 1 "Xplained_Pro_Extension_Header_2x10" H 3050 2700 50  0000 C CNN
-F 2 "" H 3000 3300 50  0001 C CNN
+F 2 "Socket_Strips:Socket_Strip_Angled_2x10_Pitch2.54mm" H 3000 3300 50  0001 C CNN
 F 3 "" H 3000 3300 50  0001 C CNN
 	1    3000 3300
@@
 F 0 "J2" H 3100 5900 50  0000 C CNN
 F 1 "Xplained_Pro_Extension_Header_2x10" H 3100 4800 50  0000 C CNN
-F 2 "" H 3050 5400 50  0001 C CNN
+F 2 "Socket_Strips:Socket_Strip_Angled_2x10_Pitch2.54mm" H 3050 5400 50  0001 C CNN
 F 3 "" H 3050 5400 50  0001 C CNN
 	1    3050 5400
@@
 F 0 "J3" H 5300 6950 50  0000 C CNN
 F 1 "Xplained_Pro_Extension_Header_2x10" H 5300 5850 50  0000 C CNN
-F 2 "" H 5250 6450 50  0001 C CNN
+F 2 "Socket_Strips:Socket_Strip_Angled_2x10_Pitch2.54mm" H 5250 6450 50  0001 C CNN
 F 3 "" H 5250 6450 50  0001 C CNN
 	1    5250 6450

Commit message: add grounds
Connections:
- net GND: now reaches J1.19 (GND)
- net GND: now also J1.2 (GND), J2.19 (GND), J2.2 (GND), J3.19 (GND), J3.2 (GND)
Changed lines of the file:
@@
 LIBS:valves
 LIBS:jdk_lib
+LIBS:daughter_board-cache
 EELAYER 25 0
 EELAYER END
@@
 	1    0    0    -1
 $EndComp
+$Comp
+L GND #PWR?
+U 1 1 5AC6DD8D
+P 3650 5000
+F 0 "#PWR?" H 3650 4750 50  0001 C CNN
+F 1 "GND" H 3650 4850 50  0000 C CNN
+F 2 "" H 3650 5000 50  0001 C CNN
+F 3 "" H 3650 5000 50  0001 C CNN
+	1    3650 5000
+	0    -1   -1   0
+$EndComp
+$Comp
+L GND #PWR?
+U 1 1 5AC6DDAF
+P 2250 5900
+F 0 "#PWR?" H 2250 5650 50  0001 C CNN
+F 1 "GND" H 2250 5750 50  0000 C CNN
+F 2 "" H 2250 5900 50  0001 C CNN
+F 3 "" H 2250 5900 50  0001 C CNN
+	1    2250 5900
+	0    1    1    0
+$EndComp
+$Comp
+L GND #PWR?
+U 1 1 5AC6DDC6
+P 3650 2900
+F 0 "#PWR?" H 3650 2650 50  0001 C CNN
+F 1 "GND" H 3650 2750 50  0000 C CNN
+F 2 "" H 3650 2900 50  0001 C CNN
+F 3 "" H 3650 2900 50  0001 C CNN
+	1    3650 2900
+	0    -1   -1   0
+$EndComp
+$Comp
+L GND #PWR?
+U 1 1 5AC6DDDD
+P 2150 3800
+F 0 "#PWR?" H 2150 3550 50  0001 C CNN
+F 1 "GND" H 2150 3650 50  0000 C CNN
+F 2 "" H 2150 3800 50  0001 C CNN
+F 3 "" H 2150 3800 50  0001 C CNN
+	1    2150 3800
+	0    1    1    0
+$EndComp
+Wire Wire Line
+	3650 2900 3450 2900
+Wire Wire Line
+	2150 3800 2600 3800
+Wire Wire Line
+	3650 5000 3500 5000
+Wire Wire Line
+	2250 5900 2650 5900
+$Comp
+L GND #PWR?
+U 1 1 5AC6DE4A
+P 5950 6050
+F 0 "#PWR?" H 5950 5800 50  0001 C CNN
+F 1 "GND" H 5950 5900 50  0000 C CNN
+F 2 "" H 5950 6050 50  0001 C CNN
+F 3 "" H 5950 6050 50  0001 C CNN
+	1    5950 6050
+	0    -1   -1   0
+$EndComp
+$Comp
+L GND #PWR?
+U 1 1 5AC6DE61
+P 4550 6950
+F 0 "#PWR?" H 4550 6700 50  0001 C CNN
+F 1 "GND" H 4550 6800 50  0000 C CNN
+F 2 "" H 4550 6950 50  0001 C CNN
+F 3 "" H 4550 6950 50  0001 C CNN
+	1    4550 6950
+	0    1    1    0
+$EndComp
+Wire Wire Line
+	5950 6050 5700 6050
+Wire Wire Line
+	4550 6950 4850 6950
 $EndSCHEMATC

Commit message: Wire ms5611
ms5611 wired for twi interface with address 0x76
Parts:
- added C1: 100nF, symbol C
- U1: footprint Housings_LGA:LGA-8_3x5mm_Pitch1.25mm -> (none)
Connections:
- net labels added: +3.3V, TWI_SCL, TWI_SDA
- wire segments 6 -> 27
Other:
- note added: "twi address is 0x76 because csb is low \n(would be 0x77 if csb was high)"
Changed lines of the file:
@@
 $EndDescr
-$Comp
-L ms5611 U1
-U 1 1 5AB44851
-P 5550 3600
-F 0 "U1" H 5975 3100 60  0000 C CNN
-F 1 "ms5611" H 5550 3600 60  0000 C CNN
-F 2 "Housings_LGA:LGA-8_3x5mm_Pitch1.25mm" H 5575 3725 60  0001 C CNN
-F 3 "" H 5575 3725 60  0001 C CNN
-	1    5550 3600
-	1    0    0    -1
-$EndComp
 $Comp
 L Xplained_Pro_Extension_Header_2x10 J1
@@
 $EndComp
 $Comp
-L GND #PWR?
+L GND #PWR4
 U 1 1 5AC6DD8D
 P 3650 5000
-F 0 "#PWR?" H 3650 4750 50  0001 C CNN
+F 0 "#PWR4" H 3650 4750 50  0001 C CNN
 F 1 "GND" H 3650 4850 50  0000 C CNN
 F 2 "" H 3650 5000 50  0001 C CNN
@@
 $EndComp
 $Comp
-L GND #PWR?
+L GND #PWR1
 U 1 1 5AC6DDAF
 P 2250 5900
-F 0 "#PWR?" H 2250 5650 50  0001 C CNN
+F 0 "#PWR1" H 2250 5650 50  0001 C CNN
 F 1 "GND" H 2250 5750 50  0000 C CNN
 F 2 "" H 2250 5900 50  0001 C CNN
@@
 $EndComp
 $Comp
-L GND #PWR?
+L GND #PWR3
 U 1 1 5AC6DDC6
 P 3650 2900
-F 0 "#PWR?" H 3650 2650 50  0001 C CNN
+F 0 "#PWR3" H 3650 2650 50  0001 C CNN
 F 1 "GND" H 3650 2750 50  0000 C CNN
 F 2 "" H 3650 2900 50  0001 C CNN
@@
 $EndComp
 $Comp
-L GND #PWR?
+L GND #PWR2
 U 1 1 5AC6DDDD
-P 2150 3800
-F 0 "#PWR?" H 2150 3550 50  0001 C CNN
-F 1 "GND" H 2150 3650 50  0000 C CNN
-F 2 "" H 2150 3800 50  0001 C CNN
-F 3 "" H 2150 3800 50  0001 C CNN
-	1    2150 3800
+P 2300 3800
+F 0 "#PWR2" H 2300 3550 50  0001 C CNN
+F 1 "GND" H 2300 3650 50  0000 C CNN
+F 2 "" H 2300 3800 50  0001 C CNN
+F 3 "" H 2300 3800 50  0001 C CNN
+	1    2300 3800
 	0    1    1    0
 $EndComp
-Wire Wire Line
-	3650 2900 3450 2900
-Wire Wire Line
-	2150 3800 2600 3800
-Wire Wire Line
-	3650 5000 3500 5000
-Wire Wire Line
-	2250 5900 2650 5900
-$Comp
-L GND #PWR?
+$Comp
+L GND #PWR8
 U 1 1 5AC6DE4A
-P 5950 6050
-F 0 "#PWR?" H 5950 5800 50  0001 C CNN
-F 1 "GND" H 5950 5900 50  0000 C CNN
-F 2 "" H 5950 6050 50  0001 C CNN
-F 3 "" H 5950 6050 50  0001 C CNN
-	1    5950 6050
+P 5650 6050
+F 0 "#PWR8" H 5650 5800 50  0001 C CNN
+F 1 "GND" H 5650 5900 50  0000 C CNN
+F 2 "" H 5650 6050 50  0001 C CNN
+F 3 "" H 5650 6050 50  0001 C CNN
+	1    5650 6050
 	0    -1   -1   0
 $EndComp
 $Comp
-L GND #PWR?
+L GND #PWR5
 U 1 1 5AC6DE61
 P 4550 6950
-F 0 "#PWR?" H 4550 6700 50  0001 C CNN
+F 0 "#PWR5" H 4550 6700 50  0001 C CNN
 F 1 "GND" H 4550 6800 50  0000 C CNN
 F 2 "" H 4550 6950 50  0001 C CNN
@@
 	0    1    1    0
 $EndComp
-Wire Wire Line
-	5950 6050 5700 6050
-Wire Wire Line
-	4550 6950 4850 6950
+$Comp
+L ms5611 U1
+U 1 1 5ACD4542
+P 6300 3450
+F 0 "U1" H 6600 2950 60  0000 C CNN
+F 1 "ms5611" H 6300 3650 60  0000 C CNN
+F 2 "" H 6325 3575 60  0001 C CNN
+F 3 "" H 6325 3575 60  0001 C CNN
+	1    6300 3450
+	1    0    0    -1
+$EndComp
+$Comp
+L GND #PWR7
+U 1 1 5ACD4FC5
+P 5050 4200
+F 0 "#PWR7" H 5050 3950 50  0001 C CNN
+F 1 "GND" H 5050 4050 50  0000 C CNN
+F 2 "" H 5050 4200 50  0001 C CNN
+F 3 "" H 5050 4200 50  0001 C CNN
+	1    5050 4200
+	1    0    0    -1
+$EndComp
+Text GLabel 2500 3400 0    60   BiDi ~ 0
+TWI_SDA
+Text GLabel 3500 3400 2    60   BiDi ~ 0
+TWI_SCL
+Text GLabel 7250 3750 2    60   BiDi ~ 0
+TWI_SCL
+Text GLabel 7250 3550 2    60   BiDi ~ 0
+TWI_SDA
+$Comp
+L C C1
+U 1 1 5ACD5730
+P 5050 3750
+F 0 "C1" H 5075 3850 50  0000 L CNN
+F 1 "100nF" H 5075 3650 50  0000 L CNN
+F 2 "" H 5088 3600 50  0001 C CNN
+F 3 "" H 5050 3750 50  0001 C CNN
+	1    5050 3750
+	1    0    0    -1
+$EndComp
+$Comp
+L +3.3V #PWR6
+U 1 1 5ACD59E1
+P 5050 3200
+F 0 "#PWR6" H 5050 3050 50  0001 C CNN
+F 1 "+3.3V" H 5050 3340 50  0000 C CNN
+F 2 "" H 5050 3200 50  0001 C CNN
+F 3 "" H 5050 3200 50  0001 C CNN
+	1    5050 3200
+	1    0    0    -1
+$EndComp
+Wire Wire Line
+	2300 3800 2750 3800
+Wire Wire Line
+	3650 2900 3250 2900
+Wire Wire Line
+	3650 5000 3300 5000
+Wire Wire Line
+	2250 5900 2800 5900
+Wire Wire Line
+	4550 6950 5000 6950
+Wire Wire Line
+	5500 6050 5650 6050
+Wire Wire Line
+	5350 3350 5700 3350
+Wire Wire Line
+	5700 3150 5550 3150
+Wire Wire Line
+	5550 2950 5550 3350
+Wire Wire Line
+	5550 2950 7000 2950
+Wire Wire Line
+	7000 2950 7000 3150
+Wire Wire Line
+	7000 3150 6900 3150
+Connection ~ 5550 3350
+Connection ~ 5550 3150
+Wire Wire Line
+	5050 3550 5700 3550
+Wire Wire Line
+	5550 3550 5550 3750
+Wire Wire Line
+	5550 3750 5700 3750
+Wire Wire Line
+	2750 3400 2500 3400
+Wire Wire Line
+	3250 3400 3500 3400
+Wire Wire Line
+	6900 3750 7250 3750
+Wire Wire Line
+	6900 3550 7250 3550
+Wire Wire Line
+	5050 3200 5050 3600
+Wire Wire Line
+	5050 3900 5050 4200
+Wire Wire Line
+	5050 4000 5350 4000
+Wire Wire Line
+	5350 4000 5350 3350
+Connection ~ 5050 4000
+Connection ~ 5050 3550
+Connection ~ 5550 3550
+Text GLabel 3600 5500 2    60   BiDi ~ 0
+TWI_SCL
+Text GLabel 2500 5500 0    60   BiDi ~ 0
+TWI_SDA
+Wire Wire Line
+	2800 5500 2500 5500
+Text GLabel 5750 6550 2    60   BiDi ~ 0
+TWI_SCL
+Text GLabel 4750 6550 0    60   BiDi ~ 0
+TWI_SDA
+Wire Wire Line
+	5750 6550 5500 6550
+Wire Wire Line
+	5000 6550 4750 6550
+Text Notes 5550 4250 0    60   ~ 0
+twi address is 0x76 because csb is low \n(would be 0x77 if csb was high)
+Wire Wire Line
+	3300 5500 3600 5500
 $EndSCHEMATC

Commit message: Add ultimate gps header
only ground and 3.3V connected
Parts:
- added J?: ultimate_gps_header_1x9, symbol ultimate_gps_header_1x9
Connections:
- wire segments 27 -> 31
Changed lines of the file:
@@
+	1    0    0    -1
+$EndComp
+Text GLabel 3600 5500 2    60   BiDi ~ 0
+TWI_SCL
+Text GLabel 2500 5500 0    60   BiDi ~ 0
+TWI_SDA
+Text GLabel 5750 6550 2    60   BiDi ~ 0
+TWI_SCL
+Text GLabel 4750 6550 0    60   BiDi ~ 0
+TWI_SDA
+Text Notes 5550 4250 0    60   ~ 0
+twi address is 0x76 because csb is low \n(would be 0x77 if csb was high)
+$Comp
+L ultimate_gps_header_1x9 J?
+U 1 1 5ACD85F9
+P 9350 3700
+F 0 "J?" H 9350 4200 50  0000 C CNN
+F 1 "ultimate_gps_header_1x9" V 9500 3700 50  0000 C CNN
+F 2 "" H 9350 3700 50  0001 C CNN
+F 3 "" H 9350 3700 50  0001 C CNN
+	1    9350 3700
+	1    0    0    -1
+$EndComp
+$Comp
+L +3.3V #PWR?
+U 1 1 5ACD88ED
+P 8900 3100
+F 0 "#PWR?" H 8900 2950 50  0001 C CNN
+F 1 "+3.3V" H 8900 3240 50  0000 C CNN
+F 2 "" H 8900 3100 50  0001 C CNN
+F 3 "" H 8900 3100 50  0001 C CNN
+	1    8900 3100
+	1    0    0    -1
+$EndComp
+$Comp
+L GND #PWR?
+U 1 1 5ACD8A23
+P 8900 4300
+F 0 "#PWR?" H 8900 4050 50  0001 C CNN
+F 1 "GND" H 8900 4150 50  0000 C CNN
+F 2 "" H 8900 4300 50  0001 C CNN
+F 3 "" H 8900 4300 50  0001 C CNN
+	1    8900 4300
 	1    0    0    -1
 $EndComp
@@
 Connection ~ 5050 3550
 Connection ~ 5550 3550
-Text GLabel 3600 5500 2    60   BiDi ~ 0
-TWI_SCL
-Text GLabel 2500 5500 0    60   BiDi ~ 0
-TWI_SDA
 Wire Wire Line
 	2800 5500 2500 5500
-Text GLabel 5750 6550 2    60   BiDi ~ 0
-TWI_SCL
-Text GLabel 4750 6550 0    60   BiDi ~ 0
-TWI_SDA
 Wire Wire Line
 	5750 6550 5500 6550
 Wire Wire Line
 	5000 6550 4750 6550
-Text Notes 5550 4250 0    60   ~ 0
-twi address is 0x76 because csb is low \n(would be 0x77 if csb was high)
 Wire Wire Line
 	3300 5500 3600 5500
+Wire Wire Line
+	9150 3400 8900 3400
+Wire Wire Line
+	8900 3400 8900 3100
+Wire Wire Line
+	9150 3500 8900 3500
+Wire Wire Line
+	8900 3500 8900 4300
 $EndSCHEMATC

Commit message: Hookup ultimate gps header
Connections:
- net labels added: UART_RX, UART_TX
- wire segments 31 -> 41
Other:
- moved on the sheet: U1
Changed lines of the file:
@@
 L ms5611 U1
 U 1 1 5ACD4542
-P 6300 3450
-F 0 "U1" H 6600 2950 60  0000 C CNN
-F 1 "ms5611" H 6300 3650 60  0000 C CNN
-F 2 "" H 6325 3575 60  0001 C CNN
-F 3 "" H 6325 3575 60  0001 C CNN
-	1    6300 3450
+P 7000 2250
+F 0 "U1" H 7300 1750 60  0000 C CNN
+F 1 "ms5611" H 7000 2450 60  0000 C CNN
+F 2 "" H 7025 2375 60  0001 C CNN
+F 3 "" H 7025 2375 60  0001 C CNN
+	1    7000 2250
 	1    0    0    -1
 $EndComp
@@
 L GND #PWR7
 U 1 1 5ACD4FC5
-P 5050 4200
-F 0 "#PWR7" H 5050 3950 50  0001 C CNN
-F 1 "GND" H 5050 4050 50  0000 C CNN
-F 2 "" H 5050 4200 50  0001 C CNN
-F 3 "" H 5050 4200 50  0001 C CNN
-	1    5050 4200
+P 5750 3000
+F 0 "#PWR7" H 5750 2750 50  0001 C CNN
+F 1 "GND" H 5750 2850 50  0000 C CNN
+F 2 "" H 5750 3000 50  0001 C CNN
+F 3 "" H 5750 3000 50  0001 C CNN
+	1    5750 3000
 	1    0    0    -1
 $EndComp
-Text GLabel 2500 3400 0    60   BiDi ~ 0
-TWI_SDA
-Text GLabel 3500 3400 2    60   BiDi ~ 0
+Text GLabel 3500 3400 2    50   BiDi ~ 0
 TWI_SCL
-Text GLabel 7250 3750 2    60   BiDi ~ 0
+Text GLabel 7950 2550 2    60   BiDi ~ 0
 TWI_SCL
-Text GLabel 7250 3550 2    60   BiDi ~ 0
+Text GLabel 7950 2350 2    60   BiDi ~ 0
 TWI_SDA
 $Comp
 L C C1
 U 1 1 5ACD5730
-P 5050 3750
-F 0 "C1" H 5075 3850 50  0000 L CNN
-F 1 "100nF" H 5075 3650 50  0000 L CNN
-F 2 "" H 5088 3600 50  0001 C CNN
-F 3 "" H 5050 3750 50  0001 C CNN
-	1    5050 3750
+P 5750 2550
+F 0 "C1" H 5775 2650 50  0000 L CNN
+F 1 "100nF" H 5775 2450 50  0000 L CNN
+F 2 "" H 5788 2400 50  0001 C CNN
+F 3 "" H 5750 2550 50  0001 C CNN
+	1    5750 2550
 	1    0    0    -1
 $EndComp
@@
 L +3.3V #PWR6
 U 1 1 5ACD59E1
-P 5050 3200
-F 0 "#PWR6" H 5050 3050 50  0001 C CNN
-F 1 "+3.3V" H 5050 3340 50  0000 C CNN
-F 2 "" H 5050 3200 50  0001 C CNN
-F 3 "" H 5050 3200 50  0001 C CNN
-	1    5050 3200
+P 5750 2000
+F 0 "#PWR6" H 5750 1850 50  0001 C CNN
+F 1 "+3.3V" H 5750 2140 50  0000 C CNN
+F 2 "" H 5750 2000 50  0001 C CNN
+F 3 "" H 5750 2000 50  0001 C CNN
+	1    5750 2000
 	1    0    0    -1
 $EndComp
-Text GLabel 3600 5500 2    60   BiDi ~ 0
-TWI_SCL
-Text GLabel 2500 5500 0    60   BiDi ~ 0
+Text GLabel 2500 5500 0    50   BiDi ~ 0
 TWI_SDA
-Text GLabel 5750 6550 2    60   BiDi ~ 0
-TWI_SCL
-Text GLabel 4750 6550 0    60   BiDi ~ 0
-TWI_SDA
-Text Notes 5550 4250 0    60   ~ 0
+Text Notes 6250 3050 0    60   ~ 0
 twi address is 0x76 because csb is low \n(would be 0x77 if csb was high)
 $Comp
 L ultimate_gps_header_1x9 J?
 U 1 1 5ACD85F9
-P 9350 3700
-F 0 "J?" H 9350 4200 50  0000 C CNN
-F 1 "ultimate_gps_header_1x9" V 9500 3700 50  0000 C CNN
-F 2 "" H 9350 3700 50  0001 C CNN
-F 3 "" H 9350 3700 50  0001 C CNN
-	1    9350 3700
+P 5200 3900
+F 0 "J?" H 5200 4400 50  0000 C CNN
+F 1 "ultimate_gps_header_1x9" V 5350 3900 50  0000 C CNN
+F 2 "" H 5200 3900 50  0001 C CNN
+F 3 "" H 5200 3900 50  0001 C CNN
+	1    5200 3900
 	1    0    0    -1
 $EndComp
@@
 L +3.3V #PWR?
 U 1 1 5ACD88ED
-P 8900 3100
-F 0 "#PWR?" H 8900 2950 50  0001 C CNN
-F 1 "+3.3V" H 8900 3240 50  0000 C CNN
-F 2 "" H 8900 3100 50  0001 C CNN
-F 3 "" H 8900 3100 50  0001 C CNN
-	1    8900 3100
+P 4750 3300
+F 0 "#PWR?" H 4750 3150 50  0001 C CNN
+F 1 "+3.3V" H 4750 3440 50  0000 C CNN
+F 2 "" H 4750 3300 50  0001 C CNN
+F 3 "" H 4750 3300 50  0001 C CNN
+	1    4750 3300
 	1    0    0    -1
 $EndComp
@@
 L GND #PWR?
 U 1 1 5ACD8A23
-P 8900 4300
-F 0 "#PWR?" H 8900 4050 50  0001 C CNN
-F 1 "GND" H 8900 4150 50  0000 C CNN
-F 2 "" H 8900 4300 50  0001 C CNN
-F 3 "" H 8900 4300 50  0001 C CNN
-	1    8900 4300
+P 4750 4500
+F 0 "#PWR?" H 4750 4250 50  0001 C CNN
+F 1 "GND" H 4750 4350 50  0000 C CNN
+F 2 "" H 4750 4500 50  0001 C CNN
+F 3 "" H 4750 4500 50  0001 C CNN
+	1    4750 4500
 	1    0    0    -1
 $EndComp
@@
 	5500 6050 5650 6050
 Wire Wire Line
-	5350 3350 5700 3350
+	6050 2150 6400 2150
 Wire Wire Line
-	5700 3150 5550 3150
+	6400 1950 6250 1950
 Wire Wire Line
-	5550 2950 5550 3350
+	6250 1750 6250 2150
 Wire Wire Line
-	5550 2950 7000 2950
+	6250 1750 7700 1750
 Wire Wire Line
-	7000 2950 7000 3150
+	7700 1750 7700 1950
 Wire Wire Line
-	7000 3150 6900 3150
-Connection ~ 5550 3350
-Connection ~ 5550 3150
+	7700 1950 7600 1950
+Connection ~ 6250 2150
+Connection ~ 6250 1950
 Wire Wire Line
-	5050 3550 5700 3550
+	5750 2350 6400 2350
 Wire Wire Line
-	5550 3550 5550 3750
+	6250 2350 6250 2550
 Wire Wire Line
-	5550 3750 5700 3750
-Wire Wire Line
-	2750 3400 2500 3400
+	6250 2550 6400 2550
 Wire Wire Line
 	3250 3400 3500 3400
 Wire Wire Line
-	6900 3750 7250 3750
+	7600 2550 7950 2550
 Wire Wire Line
-	6900 3550 7250 3550
+	7600 2350 7950 2350
 Wire Wire Line
-	5050 3200 5050 3600
+	5750 2000 5750 2400
 Wire Wire Line
-	5050 3900 5050 4200
+	5750 2700 5750 3000
 Wire Wire Line
-	5050 4000 5350 4000
+	5750 2800 6050 2800
 Wire Wire Line
-	5350 4000 5350 3350
-Connection ~ 5050 4000
-Connection ~ 5050 3550
-Connection ~ 5550 3550
+	6050 2800 6050 2150
+Connection ~ 5750 2800
+Connection ~ 5750 2350
+Connection ~ 6250 2350
 Wire Wire Line
 	2800 5500 2500 5500
 Wire Wire Line
-	5750 6550 5500 6550
+	5000 3600 4750 3600
 Wire Wire Line
-	5000 6550 4750 6550
+	4750 3600 4750 3300
+Wire Wire Line
+	5000 3700 4750 3700
+Wire Wire Line
+	4750 3700 4750 4500
+Text GLabel 2500 3500 0    50   BiDi ~ 0
+UART_RX
+Wire Wire Line
+	2500 3500 2750 3500
+Text GLabel 3500 3500 2    50   BiDi ~ 0
+UART_TX
+Wire Wire Line
+	3500 3500 3250 3500
+Text GLabel 3600 5500 2    50   BiDi ~ 0
+TWI_SCL
+Text GLabel 5750 6550 2    50   BiDi ~ 0
+TWI_SCL
 Wire Wire Line
 	3300 5500 3600 5500
 Wire Wire Line
-	9150 3400 8900 3400
+	5500 6550 5750 6550
+Text GLabel 4650 6550 0    50   BiDi ~ 0
+TWI_SDA
 Wire Wire Line
-	8900 3400 8900 3100
+	5000 6550 4650 6550
+Text GLabel 2500 3400 0    50   BiDi ~ 0
+TWI_SDA
 Wire Wire Line
-	9150 3500 8900 3500
+	2750 3400 2500 3400
+Text GLabel 4650 3800 0    50   BiDi ~ 0
+UART_TX
+Text GLabel 4650 3900 0    50   BiDi ~ 0
+UART_RX
 Wire Wire Line
-	8900 3500 8900 4300
+	4650 3800 5000 3800
+Wire Wire Line
+	5000 3900 4650 3900
+Wire Wire Line
+	5000 3500 4150 3500
+Wire Wire Line
+	4150 3500 4150 3100
+Wire Wire Line
+	4150 3100 3250 3100
+Wire Wire Line
+	5000 4200 2000 4200
+Wire Wire Line
+	2000 4200 2000 3100
+Wire Wire Line
+	2000 3100 2750 3100
 $EndSCHEMATC

Commit message: Change uart global labels, add pin labels
pin labels for actual saml21 IC pins
Connections:
- net labels added: GPS_RX, GPS_TX, PA02, PA08, PA09, PB06, PB07, PB08, PB09
- net labels removed: UART_RX, UART_TX
- wire segments 41 -> 51
Other:
- moved on the sheet: J1, J2, J3, U1

Commit message: Add openlogger header to schematic
Parts:
- added J4: OpenLog_01x06, symbol OpenLog_01x06
- gave numbers to parts that had none: 1
Connections:
- net labels added: PA18, PA19, openlog_RX, openlog_TX
- wire segments 51 -> 54
Changed lines of the file:
@@
 $EndComp
 $Comp
-L GND #PWR3
+L GND #PWR6
 U 1 1 5AC6DDC6
 P 3750 1900
-F 0 "#PWR3" H 3750 1650 50  0001 C CNN
+F 0 "#PWR6" H 3750 1650 50  0001 C CNN
 F 1 "GND" H 3750 1750 50  0000 C CNN
 F 2 "" H 3750 1900 50  0001 C CNN
@@
 $EndComp
 $Comp
-L GND #PWR8
+L GND #PWR10
 U 1 1 5AC6DE4A
 P 5750 6550
-F 0 "#PWR8" H 5750 6300 50  0001 C CNN
+F 0 "#PWR10" H 5750 6300 50  0001 C CNN
 F 1 "GND" H 5750 6400 50  0000 C CNN
 F 2 "" H 5750 6550 50  0001 C CNN
@@
 $EndComp
 $Comp
-L GND #PWR5
+L GND #PWR7
 U 1 1 5AC6DE61
 P 4650 7450
-F 0 "#PWR5" H 4650 7200 50  0001 C CNN
+F 0 "#PWR7" H 4650 7200 50  0001 C CNN
 F 1 "GND" H 4650 7300 50  0000 C CNN
 F 2 "" H 4650 7450 50  0001 C CNN
@@
 $EndComp
 $Comp
-L GND #PWR7
+L GND #PWR12
 U 1 1 5ACD4FC5
 P 5850 2000
-F 0 "#PWR7" H 5850 1750 50  0001 C CNN
+F 0 "#PWR12" H 5850 1750 50  0001 C CNN
 F 1 "GND" H 5850 1850 50  0000 C CNN
 F 2 "" H 5850 2000 50  0001 C CNN
@@
 $EndComp
 $Comp
-L +3.3V #PWR6
+L +3.3V #PWR11
 U 1 1 5ACD59E1
 P 5850 1000
-F 0 "#PWR6" H 5850 850 50  0001 C CNN
+F 0 "#PWR11" H 5850 850 50  0001 C CNN
 F 1 "+3.3V" H 5850 1140 50  0000 C CNN
 F 2 "" H 5850 1000 50  0001 C CNN
@@
 twi address is 0x76 because csb is low \n(would be 0x77 if csb was high)
 $Comp
-L ultimate_gps_header_1x9 J?
+L ultimate_gps_header_1x9 J5
 U 1 1 5ACD85F9
 P 5300 2900
-F 0 "J?" H 5300 3400 50  0000 C CNN
-F 1 "ultimate_gps_header_1x9" V 5450 2900 50  0000 C CNN
+F 0 "J5" H 5300 3400 50  0000 C CNN
+F 1 "ultimate_gps_header_1x9" V 5400 2900 50  0000 C CNN
 F 2 "" H 5300 2900 50  0001 C CNN
 F 3 "" H 5300 2900 50  0001 C CNN
@@
 $EndComp
 $Comp
-L +3.3V #PWR?
+L +3.3V #PWR8
 U 1 1 5ACD88ED
 P 4850 2300
-F 0 "#PWR?" H 4850 2150 50  0001 C CNN
+F 0 "#PWR8" H 4850 2150 50  0001 C CNN
 F 1 "+3.3V" H 4850 2440 50  0000 C CNN
 F 2 "" H 4850 2300 50  0001 C CNN
@@
 $EndComp
 $Comp
-L GND #PWR?
+L GND #PWR9
 U 1 1 5ACD8A23
 P 4950 2700
-F 0 "#PWR?" H 4950 2450 50  0001 C CNN
+F 0 "#PWR9" H 4950 2450 50  0001 C CNN
 F 1 "GND" H 4950 2550 50  0000 C CNN
 F 2 "" H 4950 2700 50  0001 C CNN
@@
 Text GLabel 3700 2500 2    50   BiDi ~ 0
 GPS_RX
-Text GLabel 3600 4700 2    50   BiDi ~ 0
+Text GLabel 3700 4700 2    50   BiDi ~ 0
 TWI_SCL
 Text GLabel 5850 7050 2    50   BiDi ~ 0
@@
 	5600 6550 5750 6550
 Wire Wire Line
-	6150 1150 6350 1150
-Wire Wire Line
-	6350 1150 6500 1150
+	6150 1150 6500 1150
 Wire Wire Line
 	6500 950  6350 950
 Wire Wire Line
-	6350 750  6350 950
-Wire Wire Line
-	6350 950  6350 1150
+	6350 750  6350 1150
 Wire Wire Line
 	6350 750  7800 750
@@
 Connection ~ 6350 950
 Wire Wire Line
-	5850 1350 6350 1350
-Wire Wire Line
-	6350 1350 6500 1350
+	5850 1350 6500 1350
 Wire Wire Line
 	6350 1350 6350 1550
@@
 	7700 1350 8050 1350
 Wire Wire Line
-	5850 1000 5850 1350
-Wire Wire Line
-	5850 1350 5850 1400
-Wire Wire Line
-	5850 1700 5850 1800
-Wire Wire Line
-	5850 1800 5850 2000
+	5850 1000 5850 1400
+Wire Wire Line
+	5850 1700 5850 2000
 Wire Wire Line
 	5850 1800 6150 1800
@@
 	3700 2500 3350 2500
 Wire Wire Line
-	3300 4700 3600 4700
+	3300 4700 3700 4700
 Wire Wire Line
 	5600 7050 5850 7050
@@
 	4100 2300 3350 2300
 $Comp
-L +3.3V #PWR?
+L +3.3V #PWR5
 U 1 1 5ACDBE50
 P 3700 2800
-F 0 "#PWR?" H 3700 2650 50  0001 C CNN
+F 0 "#PWR5" H 3700 2650 50  0001 C CNN
 F 1 "+3.3V" H 3700 2940 50  0000 C CNN
 F 2 "" H 3700 2800 50  0001 C CNN
@@
 	3700 2800 3350 2800
 $Comp
-L +3.3V #PWR?
+L +3.3V #PWR3
 U 1 1 5ACDBEF9
 P 3600 5100
-F 0 "#PWR?" H 3600 4950 50  0001 C CNN
+F 0 "#PWR3" H 3600 4950 50  0001 C CNN
 F 1 "+3.3V" H 3600 5240 50  0000 C CNN
 F 2 "" H 3600 5100 50  0001 C CNN
@@
 	3600 5100 3300 5100
 $Comp
-L +3.3V #PWR?
+L +3.3V #PWR13
 U 1 1 5ACDBF7F
 P 6000 7450
-F 0 "#PWR?" H 6000 7300 50  0001 C CNN
+F 0 "#PWR13" H 6000 7300 50  0001 C CNN
 F 1 "+3.3V" H 6000 7590 50  0000 C CNN
 F 2 "" H 6000 7450 50  0001 C CNN
@@
 Text Label 2600 2500 0    50   ~ 0
 PB09
+$Comp
+L OpenLog_01x06 J4
+U 1 1 5ACDDEA5
+P 5250 4450
+F 0 "J4" H 5250 4750 50  0000 C CNN
+F 1 "OpenLog_01x06" V 5350 4400 50  0000 C CNN
+F 2 "" H 5250 4450 50  0001 C CNN
+F 3 "" H 5250 4450 50  0001 C CNN
+	1    5250 4450
+	1    0    0    -1
+$EndComp
+Text GLabel 4800 4450 0    50   BiDi ~ 0
+openlog_TX
+Wire Wire Line
+	4800 4450 5050 4450
+Text GLabel 4800 4350 0    50   BiDi ~ 0
+openlog_RX
+Wire Wire Line
+	4800 4350 5050 4350
+Text GLabel 3700 4800 2    50   BiDi ~ 0
+openlog_RX
+Wire Wire Line
+	3700 4800 3300 4800
+Text GLabel 2500 4800 0    50   BiDi ~ 0
+openlog_TX
+Wire Wire Line
+	2500 4800 2800 4800
+Text Label 3400 4700 0    50   ~ 0
+PA09
+Text Label 2550 4700 0    50   ~ 0
+PA08
+Text Label 2550 4800 0    50   ~ 0
+PA19
+Text Label 3400 4800 0    50   ~ 0
+PA18
+$Comp
+L +3.3V #PWR?
+U 1 1 5ACE0631
+P 4950 4100
+F 0 "#PWR?" H 4950 3950 50  0001 C CNN
+F 1 "+3.3V" H 4950 4240 50  0000 C CNN
+F 2 "" H 4950 4100 50  0001 C CNN
+F 3 "" H 4950 4100 50  0001 C CNN
+	1    4950 4100
+	1    0    0    -1
+$EndComp
+Wire Wire Line
+	4950 4100 4950 4550
+Wire Wire Line
+	4950 4550 5050 4550
+$Comp
+L GND #PWR?
+U 1 1 5ACE06D5
+P 4950 4900
+F 0 "#PWR?" H 4950 4650 50  0001 C CNN
+F 1 "GND" H 4950 4750 50  0000 C CNN
+F 2 "" H 4950 4900 50  0001 C CNN
+F 3 "" H 4950 4900 50  0001 C CNN
+	1    4950 4900
+	1    0    0    -1
+$EndComp
+Wire Wire Line
+	5050 4650 4950 4650
+Wire Wire Line
+	4950 4650 4950 4900
 $EndSCHEMATC
