File: daughter_board.sch (KiCad schematic (older format))
At the start: 7 parts, among them J1 Xplained_Pro_Extension_Header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, J2 Xplained_Pro_Extension_Header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, J3 Xplained_Pro_Extension_Header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, J4 OpenLog_01x06, J5 ultimate_gps_header_1x9, U1 ms5611

Commit message: Re-assign footprint to ms5611
footprint assignment got removed when ms5611 schematic symbol was removed and placed in again, this fixes that
Parts:
- U1: footprint (none) -> Housings_LGA:LGA-8_3x5mm_Pitch1.25mm
Changed lines of the file:
@@
 $EndComp
 $Comp
-L GND #PWR4
+L GND #PWR01
 U 1 1 5AC6DD8D
 P 3650 4200
-F 0 "#PWR4" H 3650 3950 50  0001 C CNN
+F 0 "#PWR01" H 3650 3950 50  0001 C CNN
 F 1 "GND" H 3650 4050 50  0000 C CNN
 F 2 "" H 3650 4200 50  0001 C CNN
@@
 $EndComp
 $Comp
-L GND #PWR1
+L GND #PWR02
 U 1 1 5AC6DDAF
 P 2250 5100
-F 0 "#PWR1" H 2250 4850 50  0001 C CNN
+F 0 "#PWR02" H 2250 4850 50  0001 C CNN
 F 1 "GND" H 2250 4950 50  0000 C CNN
 F 2 "" H 2250 5100 50  0001 C CNN
@@
 $EndComp
 $Comp
-L GND #PWR6
+L GND #PWR03
 U 1 1 5AC6DDC6
 P 3750 1900
-F 0 "#PWR6" H 3750 1650 50  0001 C CNN
+F 0 "#PWR03" H 3750 1650 50  0001 C CNN
 F 1 "GND" H 3750 1750 50  0000 C CNN
 F 2 "" H 3750 1900 50  0001 C CNN
@@
 $EndComp
 $Comp
-L GND #PWR2
+L GND #PWR04
 U 1 1 5AC6DDDD
 P 2400 2800
-F 0 "#PWR2" H 2400 2550 50  0001 C CNN
+F 0 "#PWR04" H 2400 2550 50  0001 C CNN
 F 1 "GND" H 2400 2650 50  0000 C CNN
 F 2 "" H 2400 2800 50  0001 C CNN
@@
 $EndComp
 $Comp
-L GND #PWR10
+L GND #PWR05
 U 1 1 5AC6DE4A
 P 5750 6550
-F 0 "#PWR10" H 5750 6300 50  0001 C CNN
+F 0 "#PWR05" H 5750 6300 50  0001 C CNN
 F 1 "GND" H 5750 6400 50  0000 C CNN
 F 2 "" H 5750 6550 50  0001 C CNN
@@
 $EndComp
 $Comp
-L GND #PWR7
+L GND #PWR06
 U 1 1 5AC6DE61
 P 4650 7450
-F 0 "#PWR7" H 4650 7200 50  0001 C CNN
+F 0 "#PWR06" H 4650 7200 50  0001 C CNN
 F 1 "GND" H 4650 7300 50  0000 C CNN
 F 2 "" H 4650 7450 50  0001 C CNN
@@
 F 0 "U1" H 7400 750 60  0000 C CNN
 F 1 "ms5611" H 7100 1450 60  0000 C CNN
-F 2 "" H 7125 1375 60  0001 C CNN
+F 2 "Housings_LGA:LGA-8_3x5mm_Pitch1.25mm" H 7125 1375 60  0001 C CNN
 F 3 "" H 7125 1375 60  0001 C CNN
 	1    7100 1250
@@
 $EndComp
 $Comp
-L GND #PWR12
+L GND #PWR07
 U 1 1 5ACD4FC5
 P 5850 2000
-F 0 "#PWR12" H 5850 1750 50  0001 C CNN
+F 0 "#PWR07" H 5850 1750 50  0001 C CNN
 F 1 "GND" H 5850 1850 50  0000 C CNN
 F 2 "" H 5850 2000 50  0001 C CNN
@@
 $EndComp
 $Comp
-L +3.3V #PWR11
+L +3.3V #PWR08
 U 1 1 5ACD59E1
 P 5850 1000
-F 0 "#PWR11" H 5850 850 50  0001 C CNN
+F 0 "#PWR08" H 5850 850 50  0001 C CNN
 F 1 "+3.3V" H 5850 1140 50  0000 C CNN
 F 2 "" H 5850 1000 50  0001 C CNN
@@
 $EndComp
 $Comp
-L +3.3V #PWR8
+L +3.3V #PWR09
 U 1 1 5ACD88ED
 P 4850 2300
-F 0 "#PWR8" H 4850 2150 50  0001 C CNN
+F 0 "#PWR09" H 4850 2150 50  0001 C CNN
 F 1 "+3.3V" H 4850 2440 50  0000 C CNN
 F 2 "" H 4850 2300 50  0001 C CNN
@@
 $EndComp
 $Comp
-L GND #PWR9
+L GND #PWR010
 U 1 1 5ACD8A23
 P 4950 2700
-F 0 "#PWR9" H 4950 2450 50  0001 C CNN
+F 0 "#PWR010" H 4950 2450 50  0001 C CNN
 F 1 "GND" H 4950 2550 50  0000 C CNN
 F 2 "" H 4950 2700 50  0001 C CNN
@@
 	4100 2300 3350 2300
 $Comp
-L +3.3V #PWR5
+L +3.3V #PWR011
 U 1 1 5ACDBE50
 P 3700 2800
-F 0 "#PWR5" H 3700 2650 50  0001 C CNN
+F 0 "#PWR011" H 3700 2650 50  0001 C CNN
 F 1 "+3.3V" H 3700 2940 50  0000 C CNN
 F 2 "" H 3700 2800 50  0001 C CNN
@@
 	3700 2800 3350 2800
 $Comp
-L +3.3V #PWR3
+L +3.3V #PWR012
 U 1 1 5ACDBEF9
 P 3600 5100
-F 0 "#PWR3" H 3600 4950 50  0001 C CNN
+F 0 "#PWR012" H 3600 4950 50  0001 C CNN
 F 1 "+3.3V" H 3600 5240 50  0000 C CNN
 F 2 "" H 3600 5100 50  0001 C CNN
@@
 	3600 5100 3300 5100
 $Comp
-L +3.3V #PWR13
+L +3.3V #PWR013
 U 1 1 5ACDBF7F
 P 6000 7450
-F 0 "#PWR13" H 6000 7300 50  0001 C CNN
+F 0 "#PWR013" H 6000 7300 50  0001 C CNN
 F 1 "+3.3V" H 6000 7590 50  0000 C CNN
 F 2 "" H 6000 7450 50  0001 C CNN
@@
 PA18
 $Comp
-L +3.3V #PWR?
+L +3.3V #PWR014
 U 1 1 5ACE0631
 P 4950 4100
-F 0 "#PWR?" H 4950 3950 50  0001 C CNN
+F 0 "#PWR014" H 4950 3950 50  0001 C CNN
 F 1 "+3.3V" H 4950 4240 50  0000 C CNN
 F 2 "" H 4950 4100 50  0001 C CNN
@@
 	4950 4550 5050 4550
 $Comp
-L GND #PWR?
+L GND #PWR015
 U 1 1 5ACE06D5
 P 4950 4900
-F 0 "#PWR?" H 4950 4650 50  0001 C CNN
+F 0 "#PWR015" H 4950 4650 50  0001 C CNN
 F 1 "GND" H 4950 4750 50  0000 C CNN
 F 2 "" H 4950 4900 50  0001 C CNN
