File: daughter_board.sch (KiCad schematic (older format))
At the start: 7 parts, among them J1 Xplained_Pro_Extension_Header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, J2 Xplained_Pro_Extension_Header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, J3 Xplained_Pro_Extension_Header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, J4 OpenLog_01x06, J5 ultimate_gps_header_1x9, U1 ms5611

Commit message: Assign pcb footprints
capacitor, 2 headers
Parts:
- C1: footprint (none) -> Capacitors_SMD:C_1206_HandSoldering
- J4: footprint (none) -> Socket_Strips:Socket_Strip_Straight_1x06_Pitch2.54mm
- J5: footprint (none) -> Socket_Strips:Socket_Strip_Straight_1x09_Pitch2.54mm
Changed lines of the file:
@@
 F 0 "C1" H 5875 1650 50  0000 L CNN
 F 1 "100nF" H 5875 1450 50  0000 L CNN
-F 2 "" H 5888 1400 50  0001 C CNN
+F 2 "Capacitors_SMD:C_1206_HandSoldering" H 5888 1400 50  0001 C CNN
 F 3 "" H 5850 1550 50  0001 C CNN
 	1    5850 1550
@@
 F 0 "J5" H 5300 3400 50  0000 C CNN
 F 1 "ultimate_gps_header_1x9" V 5400 2900 50  0000 C CNN
-F 2 "" H 5300 2900 50  0001 C CNN
+F 2 "Socket_Strips:Socket_Strip_Straight_1x09_Pitch2.54mm" H 5300 2900 50  0001 C CNN
 F 3 "" H 5300 2900 50  0001 C CNN
 	1    5300 2900
@@
 F 0 "J4" H 5250 4750 50  0000 C CNN
 F 1 "OpenLog_01x06" V 5350 4400 50  0000 C CNN
-F 2 "" H 5250 4450 50  0001 C CNN
+F 2 "Socket_Strips:Socket_Strip_Straight_1x06_Pitch2.54mm" H 5250 4450 50  0001 C CNN
 F 3 "" H 5250 4450 50  0001 C CNN
 	1    5250 4450

Commit message: Add Xbee header to schematic
Parts:
- added U?: XBee_Header, symbol XBee_Header
Connections:
- wire segments 54 -> 59
Other:
- moved on the sheet: J1, J2, J3, U1

Commit message: Add Xbee header and connect spi pins
Connections:
- net labels added: SPI5_MISO, SPI5_MOSI, SPI5_SCK, SPI5_SS_A
- wire segments 59 -> 67
Changed lines of the file:
@@
-$EndComp
-$Comp
-L Xplained_Pro_Extension_Header_2x10 J2
-U 1 1 5AB44C00
-P 2600 4600
-F 0 "J2" H 2650 5100 50  0000 C CNN
-F 1 "Xplained_Pro_Extension_Header_2x10" H 2650 4000 50  0000 C CNN
-F 2 "Socket_Strips:Socket_Strip_Angled_2x10_Pitch2.54mm" H 2600 4600 50  0001 C CNN
-F 3 "" H 2600 4600 50  0001 C CNN
-	1    2600 4600
-	1    0    0    -1
 $EndComp
 $Comp
@@
 L GND #PWR02
 U 1 1 5AC6DDAF
-P 1800 5100
-F 0 "#PWR02" H 1800 4850 50  0001 C CNN
-F 1 "GND" H 1800 4950 50  0000 C CNN
-F 2 "" H 1800 5100 50  0001 C CNN
-F 3 "" H 1800 5100 50  0001 C CNN
-	1    1800 5100
+P 2250 5100
+F 0 "#PWR02" H 2250 4850 50  0001 C CNN
+F 1 "GND" H 2250 4950 50  0000 C CNN
+F 2 "" H 2250 5100 50  0001 C CNN
+F 3 "" H 2250 5100 50  0001 C CNN
+	1    2250 5100
 	0    1    1    0
 $EndComp
@@
 Text GLabel 2100 2400 0    50   BiDi ~ 0
 TWI_SDA
-Wire Wire Line
-	1950 2800 2400 2800
-Wire Wire Line
-	3300 1900 2900 1900
-Wire Wire Line
-	3200 4200 2850 4200
-Wire Wire Line
-	1800 5100 2350 5100
-Wire Wire Line
-	1750 7450 2200 7450
-Wire Wire Line
-	2700 6550 2850 6550
-Wire Wire Line
-	5700 1150 5900 1150
-Wire Wire Line
-	5900 1150 6050 1150
-Wire Wire Line
-	6050 950  5900 950
-Wire Wire Line
-	5900 750  5900 950
-Wire Wire Line
-	5900 950  5900 1150
-Wire Wire Line
-	5900 750  7350 750
-Wire Wire Line
-	7350 750  7350 950
-Wire Wire Line
-	7350 950  7250 950
-Connection ~ 5900 1150
-Connection ~ 5900 950
-Wire Wire Line
-	5400 1350 5900 1350
-Wire Wire Line
-	5900 1350 6050 1350
-Wire Wire Line
-	5900 1350 5900 1550
-Wire Wire Line
-	5900 1550 6050 1550
-Wire Wire Line
-	2900 2400 3250 2400
-Wire Wire Line
-	7250 1550 7600 1550
-Wire Wire Line
-	7250 1350 7600 1350
-Wire Wire Line
-	5400 1000 5400 1350
-Wire Wire Line
-	5400 1350 5400 1400
-Wire Wire Line
-	5400 1700 5400 1800
-Wire Wire Line
-	5400 1800 5400 2000
-Wire Wire Line
-	5400 1800 5700 1800
-Wire Wire Line
-	5700 1800 5700 1150
-Connection ~ 5400 1800
-Connection ~ 5400 1350
-Connection ~ 5900 1350
-Wire Wire Line
-	2350 4700 2050 4700
-Wire Wire Line
-	2100 2500 2400 2500
-Wire Wire Line
-	3250 2500 2900 2500
-Wire Wire Line
-	2850 4700 3250 4700
-Wire Wire Line
-	2700 7050 2950 7050
-Wire Wire Line
-	2200 7050 1850 7050
-Wire Wire Line
-	2400 2400 2100 2400
-Wire Wire Line
-	4650 2500 3800 2500
-Wire Wire Line
-	3800 2500 3800 2100
-Wire Wire Line
-	3800 2100 2900 2100
-Wire Wire Line
-	4650 3200 1650 3200
-Wire Wire Line
-	1650 3200 1650 2100
-Wire Wire Line
-	1650 2100 2400 2100
-Wire Wire Line
-	4650 3000 3650 3000
-Wire Wire Line
-	3650 3000 3650 2300
-Wire Wire Line
-	3650 2300 2900 2300
 $Comp
 L +3.3V #PWR011
@@
 	1    0    0    -1
 $EndComp
-Wire Wire Line
-	3250 2800 2900 2800
 $Comp
 L +3.3V #PWR012
 U 1 1 5ACDBEF9
-P 3150 5100
-F 0 "#PWR012" H 3150 4950 50  0001 C CNN
-F 1 "+3.3V" H 3150 5240 50  0000 C CNN
-F 2 "" H 3150 5100 50  0001 C CNN
-F 3 "" H 3150 5100 50  0001 C CNN
-	1    3150 5100
-	1    0    0    -1
-$EndComp
-Wire Wire Line
-	3150 5100 2850 5100
+P 3150 4150
+F 0 "#PWR012" H 3150 4000 50  0001 C CNN
+F 1 "+3.3V" H 3150 4290 50  0000 C CNN
+F 2 "" H 3150 4150 50  0001 C CNN
+F 3 "" H 3150 4150 50  0001 C CNN
+	1    3150 4150
+	1    0    0    -1
+$EndComp
 $Comp
 L +3.3V #PWR013
@@
 	1    0    0    -1
 $EndComp
-Wire Wire Line
-	3100 7450 2700 7450
 Text GLabel 4250 2800 0    50   BiDi ~ 0
 GPS_RX
-Wire Wire Line
-	4250 2800 4650 2800
 Text GLabel 4250 2900 0    50   BiDi ~ 0
 GPS_TX
-Wire Wire Line
-	4250 2900 4650 2900
-Wire Wire Line
-	4650 2600 4400 2600
-Wire Wire Line
-	4400 2600 4400 2300
-Wire Wire Line
-	4500 2700 4650 2700
 Text Label 2150 2100 0    50   ~ 0
 PB06
@@
 Text GLabel 4100 4300 0    50   BiDi ~ 0
 openlog_TX
-Wire Wire Line
-	4100 4300 4350 4300
 Text GLabel 4100 4200 0    50   BiDi ~ 0
 openlog_RX
-Wire Wire Line
-	4100 4200 4350 4200
 Text GLabel 3250 4800 2    50   BiDi ~ 0
 openlog_RX
-Wire Wire Line
-	3250 4800 2850 4800
 Text GLabel 2050 4800 0    50   BiDi ~ 0
 openlog_TX
-Wire Wire Line
-	2050 4800 2350 4800
 Text Label 2950 4700 0    50   ~ 0
 PA09
@@
 	1    0    0    -1
 $EndComp
-Wire Wire Line
-	4250 4000 4250 4400
-Wire Wire Line
-	4250 4400 4350 4400
 $Comp
 L GND #PWR015
@@
 	1    0    0    -1
 $EndComp
-Wire Wire Line
-	4350 4500 4250 4500
-Wire Wire Line
-	4250 4500 4250 4700
 $Comp
 L XBee_Header U?
 U 1 1 5ACFF2DE
-P 5550 5750
-F 0 "U?" H 4950 5000 60  0000 C CNN
-F 1 "XBee_Header" H 5550 6500 60  0000 C CNN
-F 2 "" H 5300 5750 60  0000 C CNN
-F 3 "" H 5300 5750 60  0000 C CNN
-	1    5550 5750
-	1    0    0    -1
-$EndComp
+P 5500 6000
+F 0 "U?" H 4900 5250 60  0000 C CNN
+F 1 "XBee_Header" H 5500 6750 60  0000 C CNN
+F 2 "" H 5250 6000 60  0000 C CNN
+F 3 "" H 5250 6000 60  0000 C CNN
+	1    5500 6000
+	1    0    0    -1
+$EndComp
+$Comp
+L +3.3V #PWR?
+U 1 1 5AD00A19
+P 4600 5250
+F 0 "#PWR?" H 4600 5100 50  0001 C CNN
+F 1 "+3.3V" H 4600 5390 50  0000 C CNN
+F 2 "" H 4600 5250 50  0001 C CNN
+F 3 "" H 4600 5250 50  0001 C CNN
+	1    4600 5250
+	1    0    0    -1
+$EndComp
+$Comp
+L GND #PWR?
+U 1 1 5AD00AE8
+P 4600 6700
+F 0 "#PWR?" H 4600 6450 50  0001 C CNN
+F 1 "GND" H 4600 6550 50  0000 C CNN
+F 2 "" H 4600 6700 50  0001 C CNN
+F 3 "" H 4600 6700 50  0001 C CNN
+	1    4600 6700
+	1    0    0    -1
+$EndComp
+Wire Wire Line
+	1950 2800 2400 2800
+Wire Wire Line
+	3300 1900 2900 1900
+Wire Wire Line
+	2250 5100 2350 5100
+Wire Wire Line
+	1750 7450 2200 7450
+Wire Wire Line
+	2700 6550 2850 6550
+Wire Wire Line
+	5700 1150 6050 1150
+Wire Wire Line
+	6050 950  5900 950
+Wire Wire Line
+	5900 750  5900 1150
+Wire Wire Line
+	5900 750  7350 750
+Wire Wire Line
+	7350 750  7350 950
+Wire Wire Line
+	7350 950  7250 950
+Connection ~ 5900 1150
+Connection ~ 5900 950
+Wire Wire Line
+	5400 1350 6050 1350
+Wire Wire Line
+	5900 1350 5900 1550
+Wire Wire Line
+	5900 1550 6050 1550
+Wire Wire Line
+	2900 2400 3250 2400
+Wire Wire Line
+	7250 1550 7600 1550
+Wire Wire Line
+	7250 1350 7600 1350
+Wire Wire Line
+	5400 1000 5400 1400
+Wire Wire Line
+	5400 1700 5400 2000
+Wire Wire Line
+	5400 1800 5700 1800
+Wire Wire Line
+	5700 1800 5700 1150
+Connection ~ 5400 1800
+Connection ~ 5400 1350
+Connection ~ 5900 1350
+Wire Wire Line
+	2350 4700 2050 4700
+Wire Wire Line
+	2100 2500 2400 2500
+Wire Wire Line
+	3250 2500 2900 2500
+Wire Wire Line
+	2850 4700 3250 4700
+Wire Wire Line
+	2700 7050 2950 7050
+Wire Wire Line
+	2200 7050 1850 7050
+Wire Wire Line
+	2400 2400 2100 2400
+Wire Wire Line
+	4650 2500 3800 2500
+Wire Wire Line
+	3800 2500 3800 2100
+Wire Wire Line
+	3800 2100 2900 2100
+Wire Wire Line
+	4650 3200 1650 3200
+Wire Wire Line
+	1650 3200 1650 2100
+Wire Wire Line
+	1650 2100 2400 2100
+Wire Wire Line
+	4650 3000 3650 3000
+Wire Wire Line
+	3650 3000 3650 2300
+Wire Wire Line
+	3650 2300 2900 2300
+Wire Wire Line
+	3250 2800 2900 2800
+Wire Wire Line
+	3100 7450 2700 7450
+Wire Wire Line
+	4250 2800 4650 2800
+Wire Wire Line
+	4250 2900 4650 2900
+Wire Wire Line
+	4650 2600 4400 2600
+Wire Wire Line
+	4400 2600 4400 2300
+Wire Wire Line
+	4500 2700 4650 2700
+Wire Wire Line
+	4100 4300 4350 4300
+Wire Wire Line
+	4100 4200 4350 4200
+Wire Wire Line
+	3250 4800 2850 4800
+Wire Wire Line
+	2050 4800 2350 4800
+Wire Wire Line
+	4250 4000 4250 4400
+Wire Wire Line
+	4250 4400 4350 4400
+Wire Wire Line
+	4350 4500 4250 4500
+Wire Wire Line
+	4250 4500 4250 4700
+Wire Wire Line
+	4600 5250 4600 5400
+Wire Wire Line
+	4600 5400 4650 5400
+Wire Wire Line
+	4650 6600 4600 6600
+Wire Wire Line
+	4600 6600 4600 6700
+Wire Wire Line
+	6350 5400 6550 5400
+Wire Wire Line
+	6350 5900 6550 5900
+Wire Wire Line
+	6350 5800 6550 5800
+Text GLabel 2050 5000 0    50   BiDi ~ 0
+SPI5_MISO
+Wire Wire Line
+	2050 5000 2350 5000
+Text GLabel 3250 4900 2    50   BiDi ~ 0
+SPI5_MOSI
+Wire Wire Line
+	3250 4900 2850 4900
+$Comp
+L Xplained_Pro_Extension_Header_2x10 J2
+U 1 1 5AB44C00
+P 2600 4600
+F 0 "J2" H 2650 5100 50  0000 C CNN
+F 1 "Xplained_Pro_Extension_Header_2x10" H 2650 4000 50  0000 C CNN
+F 2 "Socket_Strips:Socket_Strip_Angled_2x10_Pitch2.54mm" H 2600 4600 50  0001 C CNN
+F 3 "" H 2600 4600 50  0001 C CNN
+	1    2600 4600
+	1    0    0    -1
+$EndComp
+Wire Wire Line
+	3200 4200 2850 4200
+Wire Wire Line
+	3150 4150 3150 5100
+Wire Wire Line
+	3150 5100 2850 5100
+Text GLabel 3250 5000 2    50   BiDi ~ 0
+SPI5_SCK
+Wire Wire Line
+	3250 5000 2850 5000
+Text GLabel 2050 4900 0    50   BiDi ~ 0
+SPI5_SS_A
+Wire Wire Line
+	2050 4900 2350 4900
+Text GLabel 6550 5400 2    50   BiDi ~ 0
+SPI5_MISO
+Text GLabel 6550 5900 2    50   BiDi ~ 0
+SPI5_MOSI
+Text GLabel 6550 5700 2    50   BiDi ~ 0
+SPI5_SCK
+Wire Wire Line
+	6350 5700 6550 5700
+Text GLabel 6550 5800 2    50   BiDi ~ 0
+SPI5_SS_A
 $EndSCHEMATC

Commit message: Label spi pins, add XBee reset button, add decoupling capacitors
Parts:
- added 10k1: R, symbol R
- added C2: 100nF, symbol C
- added C3: 100uF, symbol CP
- added SW1: SW_Push, symbol SW_Push
- gave numbers to parts that had none: 1
Connections:
- net labels added: PB15, PB16, PB22, PB23
- wire segments 67 -> 88

Commit message: Add XBee attention pin
Connections:
- net labels added: Xbee_attn
- wire segments 88 -> 78
Changed lines of the file:
@@
 	1    0    0    -1
 $EndComp
+$Comp
+L C C2
+U 1 1 5AD572BC
+P 3650 5850
+F 0 "C2" H 3675 5950 50  0000 L CNN
+F 1 "100nF" H 3675 5750 50  0000 L CNN
+F 2 "" H 3688 5700 50  0001 C CNN
+F 3 "" H 3650 5850 50  0001 C CNN
+	1    3650 5850
+	1    0    0    -1
+$EndComp
+Text GLabel 6550 5600 2    50   Output ~ 0
+Xbee_attn
 Wire Wire Line
 	1950 2800 2400 2800
@@
 	2700 6550 2850 6550
 Wire Wire Line
-	5700 1150 5900 1150
-Wire Wire Line
-	5900 1150 6050 1150
+	5700 1150 6050 1150
 Wire Wire Line
 	6050 950  5900 950
 Wire Wire Line
-	5900 750  5900 950
-Wire Wire Line
-	5900 950  5900 1150
+	5900 750  5900 1150
 Wire Wire Line
 	5900 750  7350 750
@@
 Connection ~ 5900 950
 Wire Wire Line
-	5400 1350 5900 1350
-Wire Wire Line
-	5900 1350 6050 1350
+	5400 1350 6050 1350
 Wire Wire Line
 	5900 1350 5900 1550
@@
 	7250 1350 7600 1350
 Wire Wire Line
-	5400 1000 5400 1350
+	5400 1000 5400 1400
 Wire Wire Line
-	5400 1350 5400 1400
-Wire Wire Line
-	5400 1700 5400 1800
-Wire Wire Line
-	5400 1800 5400 2000
+	5400 1700 5400 2000
 Wire Wire Line
 	5400 1800 5700 1800
@@
 	4250 4500 4250 4700
 Wire Wire Line
-	4600 5100 4600 5150
-Wire Wire Line
-	4600 5150 4600 5400
+	4600 5100 4600 5400
 Wire Wire Line
 	4600 5400 4650 5400
 Wire Wire Line
-	3650 6600 4000 6600
-Wire Wire Line
-	4000 6600 4250 6600
-Wire Wire Line
-	4250 6600 4600 6600
-Wire Wire Line
-	4600 6600 4650 6600
+	3650 6600 4650 6600
 Wire Wire Line
 	4600 6600 4600 6700
@@
 Connection ~ 4600 6600
 Wire Wire Line
-	4250 5550 4250 5700
-Wire Wire Line
-	4250 5700 4250 6050
+	4250 5550 4250 6050
 Wire Wire Line
 	4250 5700 4650 5700
 Connection ~ 4250 5700
 Wire Wire Line
-	4250 5250 4250 5150
+	4250 5150 4250 5250
 Wire Wire Line
-	3650 5150 4000 5150
-Wire Wire Line
-	4000 5150 4250 5150
-Wire Wire Line
-	4250 5150 4600 5150
+	3650 5150 4600 5150
 Connection ~ 4600 5150
 Wire Wire Line
@@
 	4000 6000 4000 6600
 Connection ~ 4250 6600
-$Comp
-L C C2
-U 1 1 5AD572BC
-P 3650 5850
-F 0 "C2" H 3675 5950 50  0000 L CNN
-F 1 "100nF" H 3675 5750 50  0000 L CNN
-F 2 "" H 3688 5700 50  0001 C CNN
-F 3 "" H 3650 5850 50  0001 C CNN
-	1    3650 5850
-	1    0    0    -1
-$EndComp
 Wire Wire Line
 	3650 5700 3650 5150
@@
 	3650 6000 3650 6600
 Connection ~ 4000 6600
+Wire Wire Line
+	6550 5600 6350 5600
+Text GLabel 2050 4400 0    50   Input ~ 0
+Xbee_attn
+Wire Wire Line
+	2050 4400 2350 4400
 $EndSCHEMATC
